File: day_07/ex00/ex00/button.kicad_sch (KiCad schematic)
At the start: 2 parts, among them SW1 SW_Push

Commit message: pcb done
Parts:
- R1: footprint (none) -> cao_empreintes_cheat:R_0603_1608Metric
- SW1: footprint (none) -> cao_empreintes_cheat:SW_SPST_B3U-1000P
Changed lines of the file:
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@@
       (effects (font (size 1.27 1.27)) (justify left))
     )
-    (property "Footprint" "" (id 2) (at 47.625 35.56 0)
+    (property "Footprint" "cao_empreintes_cheat:SW_SPST_B3U-1000P" (id 2) (at 47.625 35.56 0)
       (effects (font (size 1.27 1.27)) hide)
     )
@@
       (effects (font (size 1.27 1.27)) (justify right))
     )
-    (property "Footprint" "" (id 2) (at 40.767 26.67 0)
+    (property "Footprint" "cao_empreintes_cheat:R_0603_1608Metric" (id 2) (at 40.767 26.67 0)
       (effects (font (size 1.27 1.27)) hide)
     )
