File: day_07/ex00/ex00/ex00.kicad_sch (KiCad schematic)
At the start: 6 parts, among them Y1 16MHz

Commit message: empreintes
Parts:
- added H1: MountingHole, symbol ex00:MountingHole
- added J2: AVR-ISP, symbol ex00:AVR-ISP-6
- gave numbers to parts that had none: 1
Connections:
- net +5V: now also J2.2 (VCC)
- net GND: now also J2.6 (GND)
- net BUT_0: now reaches U1.1 (PD3)
- net LED_0: now reaches U1.12 (PB0)
- net LED_1: now reaches U1.13 (PB1)
- net LED_2: now reaches U1.14 (PB2)
- net LED_3: now reaches U1.15 (PB3)
- net LED_3: now also J2.4 (MOSI)
- net MISO: now reaches U1.16 (PB4)
- net MISO: now also J2.1 (MISO)
- net SCK: now reaches U1.17 (PB5)
- net SCK: now also J2.3 (SCK)
- net ~{RESET}: now reaches U1.29 (~{RESET}/PC6)
- net ~{RESET}: now also J2.5 (~{RST})
- net MCU_RX: now reaches U1.30 (PD0)
- net MCU_TX: now reaches U1.31 (PD1)
- net XTAL1: now reaches C2.1, U1.7 (XTAL1/PB6), Y1.3
- net XTAL2: now reaches C1.1, U1.8 (XTAL2/PB7), Y1.1
Other:
- removed sheet Untitled Sheet
- added sheet button_but0 (button.kicad_sch)
- added sheet button_reset (button.kicad_sch)
- added sheet led_0 (led.kicad_sch)
- added sheet led_1 (led.kicad_sch)
- added sheet led_2 (led.kicad_sch)
- added sheet led_3 (led.kicad_sch)
- added sheet usb flasher (usb_flasher.kicad_sch)

Commit message: pcb done
Parts:
- C1, C2, C4, C5: footprint (none) -> cao_empreintes_cheat:C_0603_1608Metric
- H1: footprint (none) -> cao_empreintes_cheat:MountingHole_2.1mm
- J2: footprint (none) -> cao_empreintes_cheat:PinHeader_2x03_P2.54mm_Vertical
- U1: footprint Package_QFP:TQFP-32_7x7mm_P0.8mm -> cao_empreintes_cheat:TQFP-32_7x7mm_P0.8mm
- Y1: footprint (none) -> cao_empreintes_cheat:Crystal_SMD_3225-4Pin_3.2x2.5mm
Connections:
- net LED_3 renamed LED_3/MOSI
