File: day_07/ex00/ex00/led.kicad_sch (KiCad schematic)
At the start: 2 parts

Commit message: pcb done
Parts:
- D4: renamed from D1; footprint (none) -> cao_empreintes_cheat:LED_0603_1608Metric
- R6: renamed from R3; footprint (none) -> cao_empreintes_cheat:R_0603_1608Metric
Changed lines of the file:
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@@
   (symbol (lib_id "Device:LED_Filled") (at 36.195 24.13 180)
     (in_bom yes) (on_board yes)
-    (property "Reference" "D1" (id 0) (at 36.195 20.955 0))
+    (property "Reference" "D4" (id 0) (at 36.195 20.955 0))
     (property "Value" "LED_Filled" (id 1) (at 41.275 27.94 0))
-    (property "Footprint" "" (id 2) (at 36.195 24.13 0)
+    (property "Footprint" "cao_empreintes_cheat:LED_0603_1608Metric" (id 2) (at 36.195 24.13 0)
       (effects (font (size 1.27 1.27)) hide)
     )
@@
   (symbol (lib_id "ex00:Resistance") (at 51.435 24.13 180)
     (in_bom yes) (on_board yes)
-    (property "Reference" "R3" (id 0) (at 51.435 19.685 0))
+    (property "Reference" "R6" (id 0) (at 51.435 19.685 0))
     (property "Value" "330R" (id 1) (at 51.435 21.59 0))
-    (property "Footprint" "" (id 2) (at 51.435 25.908 0)
+    (property "Footprint" "cao_empreintes_cheat:R_0603_1608Metric" (id 2) (at 51.435 25.908 0)
       (effects (font (size 1.27 1.27)) hide)
     )
