File: day_07/ex00/ex00/usb_flasher.kicad_sch (KiCad schematic)
At the start: 2 parts, among them J1 Conn_01x06

Commit message: pcb done
Parts:
- C3: footprint (none) -> cao_empreintes_cheat:C_0603_1608Metric
- J1: footprint (none) -> cao_empreintes_cheat:PinHeader_1x06_P2.54mm_Vertical
Changed lines of the file:
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@@
     (property "Reference" "J1" (id 0) (at 34.29 49.53 0))
     (property "Value" "Conn_01x06" (id 1) (at 31.75 41.275 90))
-    (property "Footprint" "" (id 2) (at 34.29 38.735 0)
+    (property "Footprint" "cao_empreintes_cheat:PinHeader_1x06_P2.54mm_Vertical" (id 2) (at 34.29 38.735 0)
       (effects (font (size 1.27 1.27)) hide)
     )
@@
     (property "Reference" "C3" (id 0) (at 42.545 46.99 90))
     (property "Value" "100nF" (id 1) (at 47.625 46.99 90))
-    (property "Footprint" "" (id 2) (at 41.91 43.815 0)
+    (property "Footprint" "cao_empreintes_cheat:C_0603_1608Metric" (id 2) (at 41.91 43.815 0)
       (effects (font (size 1.27 1.27)) hide)
     )
