File: day_07/ex00/ex00/ex00.kicad_pcb (KiCad board)
At the start: 2 copper layers, 22 parts, among them J1 Conn_01x06, J2 AVR-ISP, SW1 SW_Push, SW2 SW_Push, U1 ATmega48PV-10A, Y1 16MHz

Commit message: gbr/drl
Other:
- board outline added: 24.5 x 20.5 mm
Changed lines of the file:
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@@
     (pad_to_mask_clearance 0)
     (pcbplotparams
-      (layerselection 0x00010fc_ffffffff)
+      (layerselection 0x000d0ff_ffffffff)
       (disableapertmacros false)
       (usegerberextensions false)
@@
       (outputformat 1)
       (mirror false)
-      (drillshape 1)
+      (drillshape 0)
       (scaleselection 1)
       (outputdirectory "")
@@
     )
   )
+  (gr_rect (start 83.5 71.5) (end 59 92) (layer "Edge.Cuts") (width 0.1) (fill none))
   (segment (start 68.849 88.075) (end 69.674 88.9) (width 0.25) (layer "F.Cu") (net 1))
   (segment (start 65.78 85.53) (end 65.78 86.58) (width 0.25) (layer "F.Cu") (net 1))
